File: Medicion_Trifasica/Tension/Tension.kicad_sch (KiCad schematic)
At the start: 22 parts, among them IC1 ADR130BUJZ-REEL7, J1 Screw_Terminal_01x02, J2 Conn_01x02_Pin, J3 Conn_01x03_Pin, T1 Transformer_220/9, U1 LM358

Commit message: Reconexión de la PCB, y terminación de conexiones
Parts:
- removed C8: 470 uF, Capacitor_SMD:C_0402_1005Metric_Pad0.74x0.62mm_HandSolder, symbol Device:C
- removed FL1: Choke_CommonMode_FerriteCore_1234, Inductor_THT:Choke_EPCOS_B82722A, symbol Filter:Choke_CommonMode_FerriteCore_1234
Connections:
- net AC+: now also J1.1 (Pin_1); no longer J1.2 (Pin_2)
- net AC-: now also J1.2 (Pin_2); no longer J1.1 (Pin_1)
- net Input_+9V: now also C5.2, L1.1
- net Input_-9V: now also C7.2, L2.2
Other:
- moved on the sheet: J1
Changed lines of the file:
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@@
-	)
-	(junction
-		(at 205.74 114.3)
-		(diameter 0)
-		(color 0 0 0 0)
 	)
 	(junction
@@
 	)
 	(junction
-		(at 205.74 121.92)
-		(diameter 0)
-		(color 0 0 0 0)
-	)
-	(junction
 		(at 237.49 125.73)
 		(diameter 0)
@@
 	(wire
 		(pts
+			(xy 40.64 62.23) (xy 40.64 66.04)
+		)
+		(stroke
+			(width 0)
+			(type default)
+		)
+	)
+	(wire
+		(pts
 			(xy 218.44 125.73) (xy 227.33 125.73)
 		)
@@
 	(wire
 		(pts
-			(xy 208.28 121.92) (xy 208.28 120.65)
-		)
-		(stroke
-			(width 0)
-			(type default)
-		)
-	)
-	(wire
-		(pts
 			(xy 71.12 46.99) (xy 71.12 49.53)
 		)
@@
 	(wire
 		(pts
-			(xy 40.64 62.23) (xy 40.64 66.04)
-		)
-		(stroke
-			(width 0)
-			(type default)
-		)
-	)
-	(wire
-		(pts
 			(xy 97.79 55.88) (xy 100.33 55.88)
 		)
@@
 	(wire
 		(pts
-			(xy 200.66 121.92) (xy 205.74 121.92)
-		)
-		(stroke
-			(width 0)
-			(type default)
-		)
-	)
-	(wire
-		(pts
-			(xy 218.44 120.65) (xy 218.44 125.73)
+			(xy 218.44 121.92) (xy 218.44 125.73)
 		)
 		(stroke
@@
 	(wire
 		(pts
-			(xy 200.66 114.3) (xy 205.74 114.3)
-		)
-		(stroke
-			(width 0)
-			(type default)
-		)
-	)
-	(wire
-		(pts
 			(xy 71.12 53.34) (xy 72.39 53.34)
 		)
@@
 	(wire
 		(pts
-			(xy 218.44 115.57) (xy 218.44 110.49)
+			(xy 218.44 114.3) (xy 218.44 110.49)
 		)
 		(stroke
@@
 	(wire
 		(pts
-			(xy 205.74 114.3) (xy 208.28 114.3)
-		)
-		(stroke
-			(width 0)
-			(type default)
-		)
-	)
-	(wire
-		(pts
-			(xy 205.74 121.92) (xy 208.28 121.92)
-		)
-		(stroke
-			(width 0)
-			(type default)
-		)
-	)
-	(wire
-		(pts
-			(xy 208.28 114.3) (xy 208.28 115.57)
+			(xy 200.66 114.3) (xy 218.44 114.3)
+		)
+		(stroke
+			(width 0)
+			(type default)
+		)
+	)
+	(wire
+		(pts
+			(xy 200.66 121.92) (xy 218.44 121.92)
 		)
 		(stroke
@@
 	(symbol
 		(lib_id "Connector:Screw_Terminal_01x02")
-		(at 35.56 62.23 180)
+		(at 35.56 59.69 0)
+		(mirror y)
 		(unit 1)
 		(exclude_from_sim no)
@@
 		(dnp no)
 		(property "Reference" "J1"
-			(at 35.814 56.388 0)
+			(at 35.814 65.532 0)
 			(effects
 				(font
@@
 		)
 		(property "Value" "Screw_Terminal_01x02"
-			(at 35.56 55.88 0)
+			(at 35.56 66.04 0)
 			(effects
 				(font
@@
 		)
 		(property "Footprint" "TerminalBlock:TerminalBlock_bornier-2_P5.08mm"
-			(at 35.56 62.23 0)
+			(at 35.56 59.69 0)
 			(effects
 				(font
@@
 		)
 		(property "Datasheet" "~"
-			(at 35.56 62.23 0)
+			(at 35.56 59.69 0)
 			(effects
 				(font
@@
 		)
 		(property "Description" "Generic screw terminal, single row, 01x02, script generated (kicad-library-utils/schlib/autogen/connector/)"
-			(at 35.56 62.23 0)
+			(at 35.56 59.69 0)
 			(effects
 				(font
@@
 	)
 	(symbol
-		(lib_id "Device:C")
-		(at 205.74 118.11 0)
-		(unit 1)
-		(exclude_from_sim no)
-		(in_bom yes)
-		(on_board yes)
-		(dnp no)
-		(property "Reference" "C8"
-			(at 202.438 115.824 0)
-			(effects
-				(font
-					(size 1.27 1.27)
-				)
-				(justify left)
-			)
-		)
-		(property "Value" "470 uF"
-			(at 209.55 119.3799 0)
-			(effects
-				(font
-					(size 1.27 1.27)
-				)
-				(justify left)
-				(hide yes)
-			)
-		)
-		(property "Footprint" "Capacitor_SMD:C_0402_1005Metric_Pad0.74x0.62mm_HandSolder"
-			(at 206.7052 121.92 0)
-			(effects
-				(font
-					(size 1.27 1.27)
-				)
-				(hide yes)
-			)
-		)
-		(property "Datasheet" "~"
-			(at 205.74 118.11 0)
-			(effects
-				(font
-					(size 1.27 1.27)
-				)
-				(hide yes)
-			)
-		)
-		(property "Description" "Unpolarized capacitor"
-			(at 205.74 118.11 0)
-			(effects
-				(font
-					(size 1.27 1.27)
-				)
-				(hide yes)
-			)
-		)
-		(pin "2"
-		)
-		(pin "1"
-		)
-		(instances
-			(project ""
-				(path "/402dc529-0874-4d4a-9045-def8be2165ba"
-					(reference "C8")
-					(unit 1)
-				)
-			)
-		)
-	)
-	(symbol
 		(lib_id "power:PWR_FLAG")
 		(at 246.38 125.73 180)
@@
 					(unit 1)
 				)
-			)
-		)
-	)
-	(symbol
-		(lib_id "Filter:Choke_CommonMode_FerriteCore_1234")
-		(at 213.36 118.11 0)
-		(unit 1)
-		(exclude_from_sim no)
-		(in_bom yes)
-		(on_board yes)
-		(dnp no)
-		(property "Reference" "FL1"
-			(at 213.36 113.538 0)
-			(effects
-				(font
-					(size 1.27 1.27)
-				)
-			)
-		)
-		(property "Value" "Choke_CommonMode_FerriteCore_1234"
-			(at 213.233 113.03 0)
-			(effects
-				(font
-					(size 1.27 1.27)
-				)
-				(hide yes)
-			)
-		)
-		(property "Footprint" "Inductor_THT:Choke_EPCOS_B82722A"
-			(at 213.36 124.46 0)
-			(effects
-				(font
-					(size 1.27 1.27)
-				)
-				(hide yes)
-			)
-		)
-		(property "Datasheet" "~"
-			(at 213.36 126.365 0)
-			(effects
-				(font
-					(size 1.27 1.27)
-				)
-				(hide yes)
-			)
-		)
-		(property "Description" "Generic common-mode choke, ferrite core, 1234 pin order"
-			(at 213.36 118.11 0)
-			(effects
-				(font
-					(size 1.27 1.27)
-				)
-				(hide yes)
-			)
-		)
-		(pin "2"
-		)
-		(pin "1"
-		)
-		(pin "4"
-		)
-		(pin "3"
-		)
-		(instances
-			(project ""
-				(path "/402dc529-0874-4d4a-9045-def8be2165ba"
-					(reference "FL1")
-					(unit 1)
-				)
